Commit message: spitze nose for the vessel

File: description/vessel.xacro (robot description, xacro)
@@ -39,19 +39,19 @@
         <collision name="vessel_core_collision">
             <geometry>
-                <box size="0.5 0.5 0.5"/>
+                <box size="1.2 0.8 0.4"/>
             </geometry>
         </collision>
         <visual>
             <geometry>
-                <cylinder radius="0.4" length="0.4"/>
+                <box size="0.562 0.562 0.4"/>
             </geometry>
-            <origin xyz="0.6 0 0.2" rpy="0 0 0"/>
+            <origin xyz="0.6 0 0.2" rpy="0 0 0.785398"/> <!-- rotated 45° around Y-axis -->
             <material name="blue"/>
         </visual>
-        <collision name="vessel_core_collision">
+        <collision>
             <geometry>
-                <cylinder radius="0.4" length="0.4"/>
+                <box size="0.562 0.562 0.4"/>
             </geometry>
-            <origin xyz="0.6 0 0.2" rpy="0 0 0"/>
+            <origin xyz="0.6 0 0.2" rpy="0 0 0.785398"/>
         </collision>
     </link>

Commit message: changed ship for the better

File: description/vessel.xacro (robot description, xacro)
@@ -22,6 +22,5 @@
         <color rgba="0.5 0.5 0.5 1"/>
     </material>
-    <link name="base_link">
-    </link>
+    <link name="base_link" />
     <joint name="vessel_joint" type="fixed">
         <parent link="base_link"/>
@@ -33,29 +32,77 @@
             <origin xyz="0 0 0.2" rpy="0 0 0"/>
             <geometry>
-                <box size="1.2 0.8 0.4"/>
+                <box size="1.2 0.8 0.3"/>
             </geometry>
-            <material name="blue"/>
+            <material name="white"/>
         </visual>
         <collision name="vessel_core_collision">
             <geometry>
-                <box size="1.2 0.8 0.4"/>
+                <box size="1.2 0.8 0.3"/>
             </geometry>
+            <origin xyz="0 0 0.2"/>
         </collision>
+    </link>
+    <link name="captain_room">
         <visual>
             <geometry>
-                <box size="0.562 0.562 0.4"/>
+                <box size="0.7 0.5 0.25"/>
             </geometry>
-            <origin xyz="0.6 0 0.2" rpy="0 0 0.785398"/> <!-- rotated 45° around Y-axis -->
-            <material name="blue"/>
+            <origin xyz="0 0 0" rpy="0 0 0"/>
+            <material name="orange"/>
         </visual>
         <collision>
             <geometry>
-                <box size="0.562 0.562 0.4"/>
+                <box size="0.7 0.5 0.25"/>
             </geometry>
-            <origin xyz="0.6 0 0.2" rpy="0 0 0.785398"/>
+            <origin xyz="0 0 0"/>
         </collision>
     </link>
+    <joint name="captain_room_joint" type="fixed">
+        <parent link="vessel_core"/>
+        <child link="captain_room"/>
+        <origin xyz="-0.2 0 0.3" rpy="0 0 0"/>
+    </joint>
+    <link name="vessel_nose">
+        <visual>
+            <geometry>
+                <box size="0.562 0.562 0.3"/>
+            </geometry>
+            <origin xyz="0 0 0" rpy="0 0 0.785398"/>
+            <material name="white"/>
+        </visual>
+        <collision>
+            <geometry>
+                <box size="0.562 0.562 0.3"/>
+            </geometry>
+            <origin xyz="0 0 0" rpy="0 0 0.785398"/>
+        </collision>
+    </link>
+    <joint name="vessel_nose_joint" type="fixed">
+        <parent link="vessel_core"/>
+        <child link="vessel_nose"/>
+        <origin xyz="0.6 0 0.2" rpy="0 0 0"/>
+    </joint>
+    <link name="chimney">
+        <visual>
+            <geometry>
+                <cylinder radius="0.1" length="0.3"/>
+            </geometry>
+            <origin xyz="0 0 0" rpy="0 0 0"/>
+            <material name="grey"/>
+        </visual>
+        <collision>
+            <geometry>
+                <cylinder radius="0.1" length="0.3"/>
+            </geometry>
+            <origin xyz="0 0 0"/>
+        </collision>
+    </link>
+    <joint name="chimney_joint" type="fixed">
+        <parent link="vessel_core"/>
+        <child link="chimney"/>
+        <origin xyz="0.6 0 0.3" rpy="0 0 0"/>
+    </joint>
     <gazebo reference="vessel_core">
-        <material>gazebo/blue</material>
+        <material>gazebo/white</material>
     </gazebo>
 </robot>

Commit message: functioning ship with inertials and keyboard control

File: description/vessel.xacro (robot description, xacro)
@@ -76,4 +76,11 @@
             <origin xyz="0 0 0"/>
         </collision>
+        <inertial>
+            <origin xyz="0 0 0" rpy="0 0 0"/>
+            <mass value="1.0"/>
+            <inertia ixx="0.1" ixy="0.0" ixz="0.0"
+                    iyy="0.1" iyz="0.0"
+                    izz="0.1"/>
+        </inertial>
     </link>
     <joint name="captain_room_joint" type="fixed">
@@ -96,4 +103,11 @@
             <origin xyz="0 0 0" rpy="0 0 0.785398"/>
         </collision>
+        <inertial>
+            <origin xyz="0 0 0" rpy="0 0 0"/>
+            <mass value="1.0"/>
+            <inertia ixx="0.1" ixy="0.0" ixz="0.0"
+                    iyy="0.1" iyz="0.0"
+                    izz="0.1"/>
+        </inertial>
     </link>
     <joint name="vessel_nose_joint" type="fixed">
@@ -116,4 +130,11 @@
             <origin xyz="0 0 0"/>
         </collision>
+        <inertial>
+            <origin xyz="0 0 0" rpy="0 0 0"/>
+            <mass value="0.5"/>
+            <inertia ixx="0.01" ixy="0.0" ixz="0.0"
+                    iyy="0.01" iyz="0.0"
+                    izz="0.01"/>
+        </inertial>
     </link>
     <joint name="chimney_joint" type="fixed">
