Commit message: problem found! lidar works fine now

File: description/lidar.xacro (robot description, xacro)
@@ -15,5 +15,5 @@
         <collision>
             <geometry>
-                <cylinder radius="0.05" length="0.04"/>
+                <cylinder radius="0.05" length="0.01"/>
             </geometry>
         </collision>
@@ -45,5 +45,5 @@
             <plugin name="laser_controller" filename="libgazebo_ros_ray_sensor.so">
                 <ros>
-                    <argument>~/out:=scan</argument>
+                    <remap>topicName=scan</remap>
                 </ros>
                 <output_type>sensor_msgs/LaserScan</output_type>

File: description/vessel.xacro (robot description, xacro)
@@ -255,4 +255,34 @@
         <mu2>0.0001</mu2>
     </gazebo>
+    <joint name="caster_wheel_joint" type="fixed">
+        <parent link="vessel_core"/>
+        <child link="caster_wheel"/>
+        <origin xyz="0.8 0 0.12"/>
+    </joint>
+    <link name="caster_wheel">
+        <visual>
+            <geometry>
+                <sphere radius="0.1"/>
+            </geometry>
+            <material name="orange"/>
+        </visual>
+        <collision>
+            <geometry>
+                <sphere radius="0.1"/>
+            </geometry>
+        </collision>
+        <inertial>
+            <origin xyz="0 0 0" rpy="0 0 0"/>
+            <mass value="0.1"/>
+            <inertia ixx="0.01" ixy="0.0" ixz="0.0"
+                    iyy="0.01" iyz="0.0"
+                    izz="0.01"/>
+        </inertial>
+    </link>
+    <gazebo reference="caster_wheel">
+        <material>Gazebo/Orange</material>
+        <mu1>0.0001</mu1>
+        <mu2>0.0001</mu2>
+    </gazebo>
     <gazebo reference="vessel_core">
         <material>Gazebo/White</material>

Commit message: bugs and changes

File: description/lidar.xacro (robot description, xacro)
@@ -43,7 +43,7 @@
                 </range>
             </ray>
-            <plugin name="laser_controller" filename="libgazebo_ros_ray_sensor.so">
+             <plugin name="laser_controller" filename="libgazebo_ros_ray_sensor.so">
                 <ros>
-                    <remap>topicName=scan</remap>
+                    <argument>~/out:=scan</argument>
                 </ros>
                 <output_type>sensor_msgs/LaserScan</output_type>

File: description/vessel.xacro (robot description, xacro)
@@ -151,10 +151,10 @@
     </joint>
     <link name="left_wheel">
-        <visual>
+        <!-- <visual>
             <geometry>
                 <cylinder radius="0.1" length="0.05"/>
             </geometry>
             <material name="red"/>
-        </visual>
+        </visual> -->
         <collision>
             <geometry>
@@ -166,7 +166,4 @@
         </xacro:inertial_cylinder>
     </link>
-    <gazebo reference="left_wheel">
-        <material>Gazebo/Red</material>
-    </gazebo>
     <joint name="right_wheel_joint" type="continuous">
         <parent link="vessel_core"/>
@@ -177,10 +174,10 @@
     </joint>
     <link name="right_wheel">
-        <visual>
+        <!-- <visual>
             <geometry>
                 <cylinder radius="0.1" length="0.05"/>
             </geometry>
             <material name="red"/>
-        </visual>
+        </visual> -->
         <collision>
             <geometry>
@@ -192,8 +189,5 @@
         </xacro:inertial_cylinder>
     </link>
-    <gazebo reference="right_wheel">
-        <material>Gazebo/Red</material>
-    </gazebo>
-        <!-- RIGHT PROPELLER 1 -->
+        <!-- RIGHT PROPELLER -->
     <link name="right_propeller">
         <visual>
@@ -201,5 +195,4 @@
                 <cylinder radius="0.1" length="0.1"/>
             </geometry>
-            <origin xyz="0 0 0" rpy="0 0 0"/>
             <material name="blue"/>
         </visual>
@@ -208,5 +201,4 @@
                 <cylinder radius="0.1" length="0.1"/>
             </geometry>
-            <origin xyz="0 0 0"/>
         </collision>
         <xacro:inertial_cylinder mass="0.2" length="0.1" radius="0.1">
@@ -214,16 +206,15 @@
         </xacro:inertial_cylinder>
     </link>
-    <joint name="right_propeller_joint" type="continuous">
-        <parent link="vessel_core"/>  <!-- match the 'vessel_core' style you had -->
+    <joint name="right_propeller_joint" type="fixed">
+        <parent link="vessel_core"/>
         <child link="right_propeller"/>
-        <origin xyz="-0.6 -0.2 0.12" rpy="1.5708 0 1.5708"/>  <!-- from your working propeller1 -->
-        <axis xyz="0 0 1"/>
-    </joint>
-    <gazebo reference="right_propeller">
-        <material>Gazebo/Blue</material>
-        <mu1>0.0001</mu1>
-        <mu2>0.0001</mu2>
-    </gazebo>
-    <!-- LEFT PROPELLER 2 -->
+        <origin xyz="-0.6 -0.2 0.14" rpy="1.5708 0 1.5708"/> <!-- Position and rotation of the propeller -->
+    </joint>
+        <gazebo reference="right_propeller">
+            <material>Gazebo/Blue</material>
+            <mu1>0.0001</mu1>
+            <mu2>0.0001</mu2>
+        </gazebo>
+    <!-- LEFT PROPELLER -->
     <link name="left_propeller">
         <visual>
@@ -231,5 +222,4 @@
                 <cylinder radius="0.1" length="0.1"/>
             </geometry>
-            <origin xyz="0 0 0" rpy="0 0 0"/>
             <material name="blue"/>
         </visual>
@@ -238,5 +228,4 @@
                 <cylinder radius="0.1" length="0.1"/>
             </geometry>
-            <origin xyz="0 0 0"/>
         </collision>
         <xacro:inertial_cylinder mass="0.2" length="0.1" radius="0.1">
@@ -244,9 +233,8 @@
         </xacro:inertial_cylinder>
     </link>
-    <joint name="left_propeller_joint" type="continuous">
+    <joint name="left_propeller_joint" type="fixed">
         <parent link="vessel_core"/>
         <child link="left_propeller"/>
-        <origin xyz="-0.6 0.2 0.12" rpy="1.5708 0 1.5708"/>  <!-- from your working propeller2 -->
-        <axis xyz="0 0 1"/>
+        <origin xyz="-0.6 0.2 0.14" rpy="1.5708 0 1.5708"/> <!-- Position and rotation of the propeller -->
     </joint>
     <gazebo reference="left_propeller">
@@ -255,4 +243,5 @@
         <mu2>0.0001</mu2>
     </gazebo>
+    <!-- CASTER WHEEL LINK -->
     <joint name="caster_wheel_joint" type="fixed">
         <parent link="vessel_core"/>
@@ -261,10 +250,10 @@
     </joint>
     <link name="caster_wheel">
-        <visual>
+        <!-- <visual>
             <geometry>
                 <sphere radius="0.1"/>
             </geometry>
             <material name="orange"/>
-        </visual>
+        </visual> -->
         <collision>
             <geometry>
@@ -280,28 +269,34 @@
         </inertial>
     </link>
+    <gazebo reference="vessel_core">
+        <material>Gazebo/White</material>
+        <mu1>0.0001</mu1>
+        <mu2>0.0001</mu2>
+    </gazebo>
+    <gazebo reference="captain_room">
+        <material>Gazebo/Orange</material>
+        <mu1>0.0001</mu1>
+        <mu2>0.0001</mu2>
+    </gazebo>
+    <gazebo reference="vessel_nose">
+        <material>Gazebo/White</material>
+        <mu1>0.0001</mu1>
+        <mu2>0.0001</mu2>
+    </gazebo>
+    <gazebo reference="chimney">
+        <material>Gazebo/Grey</material>
+        <mu1>0.0001</mu1>
+        <mu2>0.0001</mu2>
+    </gazebo>
+    <!-- <gazebo reference="right_wheel">
+        <material>Gazebo/Red</material>
+    </gazebo>
+    <gazebo reference="left_wheel">
+        <material>Gazebo/Red</material>
+    </gazebo>
     <gazebo reference="caster_wheel">
         <material>Gazebo/Orange</material>
-        <mu1>0.0001</mu1>
-        <mu2>0.0001</mu2>
-    </gazebo>
-    <gazebo reference="vessel_core">
-        <material>Gazebo/White</material>
-        <mu1>0.0001</mu1>
-        <mu2>0.0001</mu2>
-    </gazebo>
-    <gazebo reference="captain_room">
-        <material>Gazebo/Orange</material>
-        <mu1>0.0001</mu1>
-        <mu2>0.0001</mu2>
-    </gazebo>
-    <gazebo reference="vessel_nose">
-        <material>Gazebo/White</material>
-        <mu1>0.0001</mu1>
-        <mu2>0.0001</mu2>
-    </gazebo>
-    <gazebo reference="chimney">
-        <material>Gazebo/Grey</material>
-        <mu1>0.0001</mu1>
-        <mu2>0.0001</mu2>
-    </gazebo>
+        <mu1 value = "0.001"/>
+        <mu2 value = "0.001"/>
+    </gazebo>  -->
 </robot>

Commit message: errors solved

File: description/lidar.xacro (robot description, xacro)
@@ -18,5 +18,5 @@
             </geometry>
         </collision>
-        <xacro:inertial_cylinder mass="0.1" length="0.04" radius="0.05">
+        <xacro:inertial_cylinder mass="0.1" length="0.01" radius="0.05">
             <origin xyz="0 0 0" rpy="0 0 0"/>
         </xacro:inertial_cylinder>
@@ -26,4 +26,5 @@
         <mu1>0.1</mu1>
         <mu2>0.1</mu2>
+        <self_collide>false</self_collide>
         <sensor name="laser" type="ray">
             <pose> 0 0 0 0 0 0 </pose>
@@ -32,9 +33,9 @@
             <ray>
                 <scan>
-                    <horizontal>
-                        <samples>360</samples>
-                        <min_angle>-3.14</min_angle>
-                        <max_angle>3.14</max_angle>
-                    </horizontal>
+                <horizontal>
+                    <samples>270</samples> <!-- Use 270° like a Hokuyo -->
+                    <min_angle>-2.356</min_angle> <!-- -135° -->
+                    <max_angle>2.356</max_angle>  <!-- +135° -->
+                </horizontal>
                 </scan>
                 <range>

File: description/vessel.xacro (robot description, xacro)
@@ -35,8 +35,15 @@
         <angular_damping>10.0</angular_damping>
     </link>
+    <joint name="base_footprint_joint" type="fixed">
+        <parent link="base_link"/>
+        <child link="base_footprint"/>
+        <origin xyz="0 0 0" rpy="0 0 0"/>
+    </joint>
+    <link name="base_footprint">
+    </link>
     <joint name="vessel_joint" type="fixed">
         <parent link="base_link"/>
         <child link="vessel_core"/>
-        <origin xyz="0 0 1.3" rpy="0 0 0"/>
+        <origin xyz="0 0 0" rpy="0 0 0"/>
     </joint>
     <link name="vessel_core">
@@ -97,10 +104,10 @@
             <material name="white"/>
         </visual>
-        <collision>
+        <!-- <collision>
             <geometry>
                 <box size="0.562 0.562 0.3"/>
             </geometry>
             <origin xyz="0 0 0" rpy="0 0 0.785398"/>
-        </collision>
+        </collision> -->
         <inertial>
             <origin xyz="0 0 0" rpy="0 0 0"/>
@@ -289,14 +296,14 @@
         <mu2>0.0001</mu2>
     </gazebo>
-    <!-- <gazebo reference="right_wheel">
-        <material>Gazebo/Red</material>
-    </gazebo>
-    <gazebo reference="left_wheel">
-        <material>Gazebo/Red</material>
-    </gazebo>
     <gazebo reference="caster_wheel">
         <material>Gazebo/Orange</material>
         <mu1 value = "0.001"/>
         <mu2 value = "0.001"/>
-    </gazebo>  -->
+    </gazebo>
+    <!-- <gazebo reference="right_wheel">
+        <material>Gazebo/Red</material>
+    </gazebo>
+    <gazebo reference="left_wheel">
+        <material>Gazebo/Red</material>
+    </gazebo>-->
 </robot>
