Commit message: lidar added

File: description/camera.xacro (robot description, xacro)
@@ -4,5 +4,5 @@
         <parent link="vessel_core"/>
         <child link="camera_link"/>
-        <origin xyz="1 0 0." rpy="0 0 0"/>
+        <origin xyz="1 0 0.25" rpy="0 0 0"/>
     </joint>
     <link name="camera_link">

File: description/robot.urdf.xacro (robot description, xacro)
@@ -3,4 +3,5 @@
     <xacro:include filename="vessel.xacro" />
     <xacro:include filename="camera.xacro" />
+    <xacro:include filename="lidar.xacro" />
     <xacro:include filename="gazebo_control.xacro" />
 </robot>

Commit message: tuned the rtabmap so it is funtioning, but more tuning awaited for a correct SLAM. current problem: jumpy odometry

File: description/camera.xacro (robot description, xacro)
@@ -4,5 +4,5 @@
         <parent link="vessel_core"/>
         <child link="camera_link"/>
-        <origin xyz="1 0 0.25" rpy="0 0 0"/>
+        <origin xyz="1 0 0.30" rpy="0 0 0"/>
     </joint>
     <link name="camera_link">
@@ -34,5 +34,5 @@
                 </image>
                 <clip>
-                    <near>0.05</near>
+                    <near>0.1</near>
                     <far>100</far>
                 </clip>

File: description/depth_camera.xacro (robot description, xacro)
@@ -17,5 +17,5 @@
         <parent link="depth_camera_link"/>
         <child link="depth_camera_link_optical"/>
-        <origin xyz="0 0 0" rpy="${-pi/2} 0 ${-pi/2}"/>
+        <origin xyz="0.5 0 0.2" rpy="${-pi/2} 0 ${-pi/2}"/>
     </joint>
     <link name="depth_camera_link_optical"></link>
@@ -23,9 +23,9 @@
         <material>Gazebo/Red</material>
         <sensor name="camera" type="depth">
-            <pose> 0 0 0 0 0 0 </pose>
+            <pose>1 0 0.2 0 0 0</pose> <!-- Match the optical joint offset -->
             <visualize>true</visualize>
             <update_rate>10</update_rate>
             <camera>
-                <horizontal_fov>2.0943951</horizontal_fov>
+                <horizontal_fov>1.3962634</horizontal_fov>
                 <image>
                     <width>640</width>
@@ -34,5 +34,5 @@
                 </image>
                 <clip>
-                    <near>0.05</near>
+                    <near>0.1</near>
                     <far>100</far>
                 </clip>
@@ -40,5 +40,5 @@
             <plugin name="depth_camera_controller" filename="libgazebo_ros_camera.so">
                 <frame_name>depth_camera_link_optical</frame_name>
-                <min_depth>0.05</min_depth>
+                <min_depth>0.1</min_depth>
                 <max_depth>100.0</max_depth>
             </plugin>
